File: KiCad-Files/USB-C-Hub.kicad_pcb (KiCad board)
At the start: 4 copper layers, 92.2 x 71.7 mm, 106 parts, among them J1 12401610E4#2A, J2 483930003, J3 483930003, J4 CON-SOCJ-2155, J5 Conn_01x04, J6 Conn_01x05, U1 USB5744/2G, U2 UTC2000, U3 HD3SS6126RUAR, U4 MIC2099-1YMT-TR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

Commit message: Added silkscreen and made power planes a bit wider
Parts:
- added H5: MountingHole_Pad, MountingHole:MountingHole_3mm_Pad_Via, F.Cu at (138.4, 60.0)
- added REF**: Symbol_Barrel_Polarity, Symbol:Symbol_Barrel_Polarity, F.Cu at (55.1, 86.4)
- U2: value UTC2000 -> UTC2000/MG
- moved R15 7.02 mm to (91.8, 35.4), turned to 0 degrees
- moved R12 5.90 mm to (94.5, 36.4), turned to 0 degrees
- renumbered RESET to SW1
Routing:
- net +5VD: track 103.4 -> 100.8 mm
- net GND: track 122.5 -> 124.3 mm
- net /VBUS_Host_Filt: track 73.6 -> 74.5 mm
- net +3V3: track 55.2 -> 56.0 mm
Other:
- board text added: "+"
- board text added: "-"
- board text added: "1V2"
- board text added: "3V3"
- board text added: "5V"
- board text added: "5V input"
- board text added: "GND"
- board text added: "RESET"
- board text added: "SPI_CE/ CFG_REM"
- board text added: "SPI_CLK/ SMCLK"
- board text added: "SPI_DI/ CFG_BC"
- board text added: "SPI_DO/ SMDAT"
- board text removed: "Exclusive Electronics"
