File: KiCad-Files/USB-C-Hub.kicad_sch (KiCad schematic)
At the start: 59 parts, among them J1 12401610E4#2A, J2 483930003, J3 483930003, SW1 SW_Push, U1 USB5744/2G, U2 UTC2000-I/MG, U3 HD3SS6126RUAR

Commit message: Added silkscreen and made power planes a bit wider
Parts:
- U2: value UTC2000-I/MG -> UTC2000/MG; MFR# UTC2000-E/MG -> UTC2000/MG
Connections:
- no-connect marks 30 -> 31
Changed lines of the file:
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@@
   (no_connect (at 180.34 317.5))
   (no_connect (at 468.63 240.03))
+  (no_connect (at 252.73 90.17))
   (no_connect (at 204.47 303.53))
   (no_connect (at 298.45 93.98))
@@
     (effects (font (size 1.27 1.27)) (justify left bottom))
   )
-  (text "NC pins used for straight through routing" (at 137.16 111.76 0)
+  (text "NC pins used for straight through routing" (at 138.43 128.27 0)
     (effects (font (size 1.27 1.27)) (justify left bottom))
   )
@@
   )
   (symbol (lib_id "Connector:USB3_A") (at 440.69 369.57 0) (mirror y) (unit 1)
-    (in_bom yes) (on_board yes) (fields_autoplaced)
-    (property "Reference" "J3" (id 0) (at 452.12 368.9349 0)
+    (in_bom yes) (on_board yes)
+    (property "Reference" "J3" (id 0) (at 431.8 350.52 0)
       (effects (font (size 1.27 1.27)) (justify right))
     )
-    (property "Value" "483930003" (id 1) (at 452.12 371.4749 0)
+    (property "Value" "483930003" (id 1) (at 431.8 353.06 0)
       (effects (font (size 1.27 1.27)) (justify right))
     )
@@
       (effects (font (size 1.524 1.524)))
     )
-    (property "Value" "UTC2000-I/MG" (id 1) (at 188.595 180.34 0)
+    (property "Value" "UTC2000/MG" (id 1) (at 188.595 180.34 0)
       (effects (font (size 1.524 1.524)))
     )
@@
       (effects (font (size 1.524 1.524)) hide)
     )
-    (property "Datasheet" "https://www.digikey.com/en/products/detail/microchip-technology/UTC2000-E-MG/5803607" (id 3) (at 187.96 201.93 0)
+    (property "Datasheet" "https://www.digikey.com/en/products/detail/microchip-technology/UTC2000-MG/5639492" (id 3) (at 187.96 201.93 0)
       (effects (font (size 1.524 1.524)) hide)
     )
-    (property "MFR#" "UTC2000-E/MG" (id 4) (at 189.23 201.93 0)
+    (property "MFR#" "UTC2000/MG" (id 4) (at 189.23 201.93 0)
       (effects (font (size 1.27 1.27)) hide)
     )
@@
       (reference "#PWR0108") (unit 1) (value "GND") (footprint "")
     )
+    (path "/65d11ab1-9769-4cee-9541-45d052b13890/b137e1d8-1ac8-4ec0-af77-aaf28c133529"
+      (reference "#PWR?") (unit 1) (value "GND") (footprint "")
+    )
     (path "/cfa29f6b-3d51-4474-b96b-9e793512e832"
       (reference "C1") (unit 1) (value "14pF") (footprint "Resistor_SMD:R_0402_1005Metric")
@@
       (reference "H4") (unit 1) (value "MountingHole_Pad") (footprint "MountingHole:MountingHole_3mm_Pad_Via")
     )
+    (path "/65d11ab1-9769-4cee-9541-45d052b13890/5975151e-2c1d-444c-8d6a-36206b6134f0"
+      (reference "H5") (unit 1) (value "MountingHole_Pad") (footprint "MountingHole:MountingHole_3mm_Pad_Via")
+    )
     (path "/35776aff-6edd-4fea-a89e-afaf56e80c57"
       (reference "J1") (unit 1) (value "12401610E4#2A") (footprint "Connector_USB:USB_C_Receptacle_Amphenol_12401610E4-2A")
@@
     )
     (path "/efcdadde-7a33-4c7a-9940-1f9195f8b5da"
-      (reference "U2") (unit 1) (value "UTC2000-I/MG") (footprint "UTC2000:16-pinQFN3x3")
+      (reference "U2") (unit 1) (value "UTC2000/MG") (footprint "UTC2000:16-pinQFN3x3")
     )
     (path "/02ee2d73-edc2-456b-9242-eed52c8cfe74"
